Commit message: Fixed base footprint link origin

File: install/my_rb1_description/share/my_rb1_description/urdf/my_rb1_robot.urdf (robot description, URDF)
Before this commit: robot rb1_robot, 7 links, 6 joints
Joints:
- joint base_link_plate_joint: origin xyz=0 0 0.15 rpy=0 0 0 -> xyz=0 0 0 rpy=0 0 0

Commit message: Completed task 1

File: install/my_rb1_description/share/my_rb1_description/urdf/my_rb1_robot.urdf (robot description, URDF)
Before this commit: robot rb1_robot, 7 links, 6 joints
Links:
- link back_caster: mass None -> 0.3
- link base_link: mass None -> 20.0
- link front_caster: mass None -> 0.3
- link front_laser: mass None -> 0.4; geometry collision cylinder length=0.04 radius=0.035; visual cylinder length=0.04 radius=0.035
- link left_wheel: mass None -> 2.0
- link right_wheel: mass None -> 2.0
Joints:
- joint base_link_plate_joint: origin xyz=0 0 0 rpy=0 0 0 -> xyz=0 0 0.15 rpy=0 0 0

File: my_rb1_description/urdf/my_rb1_robot.urdf (robot description, URDF)
Before this commit: robot rb1_robot, 7 links, 6 joints
Links:
- link back_caster: mass None -> 0.3
- link base_link: mass None -> 20.0
- link front_caster: mass None -> 0.3
- link front_laser: mass None -> 0.4; geometry collision cylinder length=0.04 radius=0.035; visual cylinder length=0.04 radius=0.035
- link left_wheel: mass None -> 2.0
- link right_wheel: mass None -> 2.0
